File: MainPCB/indicator_lights.kicad_sch (KiCad schematic)
At the start: 48 parts, among them Q1 AO3400A, Q2 AO3400A, Q3 AO3400A, Q4 AO3400A, U1 TLP293-4, U2 74AHCT1G125

Commit message: MCU design + global power supplies
Connections:
- net 5V renamed +5V
