File: MainPCB/mcu.kicad_sch (KiCad schematic)
At the start: 1 part, among them IC1 STM32H747IIT6

Commit message: MCU design + global power supplies
Parts:
- added C10, C11, C12, C13, C14, C15, C16, C17, C18, C19, C20, C21, C22, C23, C24, C25, C26, C27, C31, C33, C35, C38, C9: 0.1uF, symbol Device:C
- added C28, C29, C30: 2.2uF, symbol Device:C
- added C32: 1uF, symbol Device:C
- added C34: 4.7uF, symbol Device:C
- added C36, C37: 10pF, symbol Device:C
- added R17: 10k, symbol Device:R
- added Y1: 25MHz, symbol Device:Crystal
Connections:
- net PE2: now reaches IC1.1 (PE2)
- net PC14: now reaches IC1.10 (PC14-OSC32_IN)
- net GND: now reaches IC1.100 (VSS_11)
- net GND: now also IC1.101 (VCAPDSI), IC1.102 (VDD12DSI_1), IC1.105 (VSSDSI_1), IC1.108 (VDD12DSI_2), IC1.109 (VSSDSI_2), IC1.112 (VSS_12), IC1.119 (VSS_13), IC1.12 (VSS_2), IC1.134 (VSS_14), IC1.137 (VSS_15), IC1.14 (VSSSMPS), IC1.15 (VLXSMPS), IC1.151 (VSS_16), IC1.159 (VSS_17), IC1.16 (VDDSMPS), IC1.17 (VFBSMPS), IC1.173 (VSS_18), IC1.24 (VSS_3), IC1.38 (VSSA), IC1.45 (VSS_4), IC1.47 (VSS_5), IC1.6 (VSS_1), IC1.64 (VSS_6), IC1.70 (VSS_7), IC1.81 (VSS_8), IC1.83 (VSS_9), IC1.93 (VSS_10), C10.1, C11.2, C12.1, C13.2, C14.1, C15.1, C16.1, C17.1, C18.1, C19.1, C20.1, C21.1, C22.2, C23.2, C24.1, C25.1, C26.1, C27.1, C28.1, C29.1, C30.1, C31.2, C32.2, C33.1, C34.1, C35.1, C36.2, C37.2, C38.2, C9.1, R17.1
- net PC15: now reaches IC1.11 (PC15-OSC32_OUT)
- net PG2: now reaches IC1.110 (PG2)
- net PG3: now reaches IC1.111 (PG3)
- net +3V3: now reaches IC1.113 (VDD_11)
- net +3V3: now also IC1.120 (VDD50USB), IC1.121 (VDD33USB), IC1.126 (VDD_12), IC1.13 (VDD_2), IC1.135 (VDDLDO_2), IC1.136 (VDD_13), IC1.152 (VDD_14), IC1.160 (VDD_15), IC1.174 (PDR_ON), IC1.175 (VDDLDO_3), IC1.176 (VDD_16), IC1.25 (VDD_3), IC1.39 (VREF+), IC1.40 (VDDA), IC1.44 (VDD_4), IC1.48 (VDD_5), IC1.65 (VDD_6), IC1.7 (VDD_1), IC1.71 (VDD_7), IC1.8 (VBAT), IC1.82 (VDDLDO_1), IC1.84 (VDD_8), IC1.92 (VDD_9), IC1.99 (VDD_10), C10.2, C11.1, C12.2, C13.1, C14.2, C15.2, C16.2, C17.2, C18.2, C19.2, C20.2, C21.2, C22.1, C24.2, C25.2, C26.2, C27.2, C31.1, C32.1, C33.2, C34.2, C35.2, C38.1, C9.2
- net PG4: now reaches IC1.114 (PG4)
- net PG5: now reaches IC1.115 (PG5)
- net PG6: now reaches IC1.116 (PG6)
- net PG7: now reaches IC1.117 (PG7)
- net PG8: now reaches IC1.118 (PG8)
- net PC6: now reaches IC1.122 (PC6)
- net PC7: now reaches IC1.123 (PC7)
- net PC8: now reaches IC1.124 (PC8)
- net PC9: now reaches IC1.125 (PC9)
- net PA8: now reaches IC1.127 (PA8)
- net PA9: now reaches IC1.128 (PA9)
- net PA10: now reaches IC1.129 (PA10)
- net PA11: now reaches IC1.130 (PA11)
- net PA12: now reaches IC1.131 (PA12)
- net PA13: now reaches IC1.132 (PA13)
- net at IC1.133 (VCAP_2): now also C28.2
- net PA14: now reaches IC1.138 (PA14)
- net PA15: now reaches IC1.139 (PA15)
- net PC10: now reaches IC1.140 (PC10)
- net PC11: now reaches IC1.141 (PC11)
- net PC12: now reaches IC1.142 (PC12)
- net PD0: now reaches IC1.143 (PD0)
- net PD1: now reaches IC1.144 (PD1)
- net PD2: now reaches IC1.145 (PD2)
- net PD3: now reaches IC1.146 (PD3)
- net PD4: now reaches IC1.147 (PD4)
- net PD5: now reaches IC1.148 (PD5)
- net PD6: now reaches IC1.149 (PD6)
- net PD7: now reaches IC1.150 (PD7)
- net PG9: now reaches IC1.153 (PG9)
- net PG10: now reaches IC1.154 (PG10)
- net PG11: now reaches IC1.155 (PG11)
- net PG12: now reaches IC1.156 (PG12)
- net PG13: now reaches IC1.157 (PG13)
- net PG14: now reaches IC1.158 (PG14)
- net PG15: now reaches IC1.161 (PG15)
- net PB3: now reaches IC1.162 (PB3)
- net PB4: now reaches IC1.163 (PB4)
- net PB5: now reaches IC1.164 (PB5)
- net PB6: now reaches IC1.165 (PB6)
- net PB7: now reaches IC1.166 (PB7)
- net at IC1.167 (BOOT0): now also R17.2
- net PB8: now reaches IC1.168 (PB8)
- net PB9: now reaches IC1.169 (PB9)
- net PE0: now reaches IC1.170 (PE0)
- net PE1: now reaches IC1.171 (PE1)
- net at IC1.172 (VCAP_3): now also C30.2
- net PF0: now reaches IC1.18 (PF0)
- net PF1: now reaches IC1.19 (PF1)
- net PE3: now reaches IC1.2 (PE3)
- net PF2: now reaches IC1.20 (PF2)
- net PF3: now reaches IC1.21 (PF3)
- net PF4: now reaches IC1.22 (PF4)
- net PF5: now reaches IC1.23 (PF5)
- net PF6: now reaches IC1.26 (PF6)
- net PF7: now reaches IC1.27 (PF7)
- net PF8: now reaches IC1.28 (PF8)
- net PF9: now reaches IC1.29 (PF9)
- net PE4: now reaches IC1.3 (PE4)
- net PF10: now reaches IC1.30 (PF10)
- net at IC1.31 (PH0-OSC_IN): now also C36.1, Y1.1
- net at IC1.32 (PH1-OSC_OUT): now also C37.1, Y1.2
- net NRST: now reaches IC1.33 (NRST)
- net NRST: now also C23.1
- net PC0: now reaches IC1.34 (PC0)
- net PC1: now reaches IC1.35 (PC1)
- net PC2: now reaches IC1.36 (PC2_C)
- net PC3: now reaches IC1.37 (PC3_C)
- net PE5: now reaches IC1.4 (PE5)
- net PA0: now reaches IC1.41 (PA0)
- net PA1: now reaches IC1.42 (PA1)
- net PA2: now reaches IC1.43 (PA2)
- net PA3: now reaches IC1.46 (PA3)
- net PA4: now reaches IC1.49 (PA4)
- net PE6: now reaches IC1.5 (PE6)
- net PA5: now reaches IC1.50 (PA5)
- net PA6: now reaches IC1.51 (PA6)
- net PA7: now reaches IC1.52 (PA7)
- net PC4: now reaches IC1.53 (PC4)
- net PC5: now reaches IC1.54 (PC5)
- net PB0: now reaches IC1.55 (PB0)
- net PB1: now reaches IC1.56 (PB1)
- net PB2: now reaches IC1.57 (PB2)
- net PF11: now reaches IC1.58 (PF11)
- net PF12: now reaches IC1.59 (PF12)
- net PF13: now reaches IC1.60 (PF13)
- net PF14: now reaches IC1.61 (PF14)
- net PF15: now reaches IC1.62 (PF15)
- net PG0: now reaches IC1.63 (PG0)
- net PG1: now reaches IC1.66 (PG1)
- net PE7: now reaches IC1.67 (PE7)
- net PE8: now reaches IC1.68 (PE8)
- net PE9: now reaches IC1.69 (PE9)
- net PE10: now reaches IC1.72 (PE10)
- net PE11: now reaches IC1.73 (PE11)
- net PE12: now reaches IC1.74 (PE12)
- net PE13: now reaches IC1.75 (PE13)
- net PE14: now reaches IC1.76 (PE14)
- net PE15: now reaches IC1.77 (PE15)
- net PB10: now reaches IC1.78 (PB10)
- net PB11: now reaches IC1.79 (PB11)
- net at IC1.80 (VCAP_1): now also C29.2
- net PB12: now reaches IC1.85 (PB12)
- net PB13: now reaches IC1.86 (PB13)
- net PB14: now reaches IC1.87 (PB14)
- net PB15: now reaches IC1.88 (PB15)
- net PD8: now reaches IC1.89 (PD8)
- net PC13: now reaches IC1.9 (PC13)
- net PD9: now reaches IC1.90 (PD9)
- net PD10: now reaches IC1.91 (PD10)
- net PD11: now reaches IC1.94 (PD11)
- net PD12: now reaches IC1.95 (PD12)
- net PD13: now reaches IC1.96 (PD13)
- net PD14: now reaches IC1.97 (PD14)
- net PD15: now reaches IC1.98 (PD15)
- no-connect marks 0 -> 4
Other:
- moved on the sheet: IC1
